Commit message: Adiciona aplicativo acessivel, supervisao de movimento e watchdog independente

File: dog_ia/urdf/dog_ia.urdf.xacro (robot description, xacro)
@@ -46,5 +46,5 @@
   <link name="mast_link">
     <visual><geometry><box size="0.035 0.035 0.35"/></geometry><material name="silver"/></visual>
-    <collision><geometry><box size="0.035 0.035 0.35"/></geometry></collision>
+    <!-- Visual-only mast collision: avoids self-occlusion in this simplified ray model. -->
     <xacro:box_inertia m="0.2" x="0.035" y="0.035" z="0.35"/>
   </link>
@@ -88,8 +88,9 @@
   <gazebo>
     <plugin name="drive" filename="libgazebo_ros_diff_drive.so">
+      <ros><remapping>cmd_vel:=/cmd_vel_safe</remapping></ros>
       <update_rate>30</update_rate><left_joint>left_wheel_joint</left_joint><right_joint>right_wheel_joint</right_joint>
       <wheel_separation>0.39</wheel_separation><wheel_diameter>0.2</wheel_diameter>
       <max_wheel_torque>15</max_wheel_torque><max_wheel_acceleration>1.5</max_wheel_acceleration>
-      <command_topic>cmd_vel</command_topic><odometry_topic>odom</odometry_topic>
+      <command_topic>cmd_vel_safe</command_topic><odometry_topic>odom</odometry_topic>
       <odometry_frame>odom</odometry_frame><robot_base_frame>base_footprint</robot_base_frame>
       <publish_odom>true</publish_odom><publish_odom_tf>true</publish_odom_tf><publish_wheel_tf>false</publish_wheel_tf>

Commit message: Implementa percepcao controlada de semaforos e riscos 3D com voz

File: dog_ia/urdf/dog_ia.urdf.xacro (robot description, xacro)
@@ -86,4 +86,25 @@
     </sensor>
   </gazebo>
+  <link name="ground_camera_link"><visual><geometry><box size="0.05 0.08 0.04"/></geometry><material name="black"/></visual><xacro:box_inertia m="0.1" x="0.05" y="0.08" z="0.04"/></link>
+  <joint name="ground_camera_joint" type="fixed"><parent link="base_link"/><child link="ground_camera_link"/><origin xyz="0.23 0 0.2" rpy="0 0.55 0"/></joint>
+  <link name="ground_optical_frame"/>
+  <joint name="ground_optical_joint" type="fixed"><parent link="ground_camera_link"/><child link="ground_optical_frame"/><origin rpy="${-pi/2} 0 ${-pi/2}"/></joint>
+  <gazebo reference="ground_camera_link">
+    <sensor name="ground_rgbd_camera" type="depth">
+      <always_on>true</always_on><update_rate>10</update_rate>
+      <camera><horizontal_fov>1.2</horizontal_fov><image><width>320</width><height>240</height><format>R8G8B8</format></image><clip><near>0.1</near><far>8</far></clip></camera>
+      <plugin name="ground_camera_ros" filename="libgazebo_ros_camera.so">
+        <ros><namespace>/ground</namespace>
+          <remapping>rgbd/image_raw:=/ground/image_raw</remapping>
+          <remapping>rgbd/ground_info:=/ground/ground_info</remapping>
+          <remapping>rgbd/depth/image_raw:=/ground/depth/image_raw</remapping>
+          <remapping>rgbd/depth/ground_info:=/ground/depth/ground_info</remapping>
+          <remapping>rgbd/points:=/ground/points</remapping>
+        </ros>
+        <camera_name>rgbd</camera_name><frame_name>ground_optical_frame</frame_name>
+        <min_depth>0.1</min_depth><max_depth>8.0</max_depth>
+      </plugin>
+    </sensor>
+  </gazebo>
   <gazebo>
     <plugin name="drive" filename="libgazebo_ros_diff_drive.so">
